File: hardware/Main.brd (EAGLE design)
At the start: 86.4 x 49.7 mm, 90 parts, among them IC1 ESP32-WROOM-32D_M113DH3200PH3Q, IC2 LAN8720A-CP-ABC, IC3 R-78E5.0-1.0, IC4 LT1129MPST-3.3#PBF, J2 1727078, J3 HR911105A, J4 1727010, J5 1727049, J6 1727049, Q1 O50.0-JO32-B-3.3-1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

Commit message: Layout fertig
Parts:
- added C23: 100nF, rcl:C0603
- added IC5: 74LVT2244PW,118, SamacSys_Parts:SOP65P640X110-20N
Connections:
- new net N$1: IC5.18, R32.1
- new net N$10: IC5.14, R36.1
- new net N$17: IC5.12, R38.1
- new net N$32: IC5.9, R4.1
- new net N$7: IC5.16, R34.1
- net +5V: now also C23.1, IC5.20
- net GND: now also C23.2, IC5.1, IC5.10, IC5.13, IC5.15, IC5.17, IC5.19
- net REL_CH_00: now also IC5.2; no longer R32.1
- net REL_CH_01: now also IC5.4; no longer R34.1
- net REL_CH_02: now also IC5.6; no longer R36.1
- net REL_CH_03: now also IC5.8; no longer R38.1
- net REL_CH_04: now also IC5.11; no longer R4.1
Routing:
- net +5V: track 53.4 -> 91.0 mm
- net REL_CH_04: track 35.3 -> 61.1 mm, vias 2 -> 3
- net N$17: track 0.00 -> 20.5 mm, vias 0 -> 1
- net N$32: track 0.00 -> 18.0 mm, vias 0 -> 1
- net N$10: track 0.00 -> 13.6 mm, vias 0 -> 1
- net REL_CH_03: track 11.9 -> 22.2 mm, vias 0 -> 1
- net REL_CH_02: track 17.7 -> 26.5 mm, vias 0 -> 1
- net N$7: track 0.00 -> 5.67 mm, vias 0 -> 1
- net N$1: track 0.00 -> 5.55 mm, vias 0 -> 1
- net REL_CH_01: track 19.0 -> 22.8 mm, vias 0 -> 1
- net REL_CH_00: track 24.2 -> 21.6 mm, vias 0 -> 1
- net ETH_RXD0: track 40.6 -> 39.2 mm
Other:
- board text added: "+"
- board text added: "O1"
- board text added: "O2"
- board text added: "O3"
- board text added: "O4"
- board text added: "O5"
